File: SNAP Project PCB Files/PCB Files V6.0/SNAP_Project.kicad_sch (KiCad schematic)
At the start: 52 parts, among them IC1 ADP121-AUJZ30R7, J1 USB_C_Receptacle_USB2.0, J3 Serial Wire Debug, J4 OLED Screen Conn, Q1 2N7000, Q2 2N7000, Q3 2N7000, Q5 2N7002KDW_R1_00001, Q6 771-BSS84AK215, SW1 OS102011MA1QN1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

Commit message: 4v Line fix
Connections:
- net +3V0: no longer C2.1, IC1.5 (VOUT)
- net +4V: now also C2.1, IC1.5 (VOUT); no longer C1.1, D5.1 (K), IC1.1 (VIN), Q6.1 (D), SW1.1 (A), TP3.1
- new net VDD: C1.1, D5.1 (K), IC1.1 (VIN), Q6.1 (D), SW1.1 (A), TP3.1
Other:
- moved on the sheet: TP3
Changed lines of the file:
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@@
   (junction (at 68.58 41.275) (diameter 0) (color 0 0 0 0)
   )
+  (junction (at 27.94 132.08) (diameter 0) (color 0 0 0 0)
+  )
   (junction (at 135.255 171.45) (diameter 0) (color 0 0 0 0)
   )
@@
   (junction (at 248.92 57.15) (diameter 0) (color 0 0 0 0)
   )
-  (junction (at 281.305 57.15) (diameter 0) (color 0 0 0 0)
+  (junction (at 281.94 57.15) (diameter 0) (color 0 0 0 0)
   )
   (junction (at 120.65 187.96) (diameter 0) (color 0 0 0 0)
@@
   )
   (junction (at 38.1 131.445) (diameter 0) (color 0 0 0 0)
-  )
-  (junction (at 27.94 131.445) (diameter 0) (color 0 0 0 0)
   )
   (junction (at 265.43 34.925) (diameter 0) (color 0 0 0 0)
@@
     (stroke (width 0) (type default) (color 0 0 0 0))
   )
+  (wire (pts (xy 22.86 125.73) (xy 22.86 132.08))
+    (stroke (width 0) (type default) (color 0 0 0 0))
+  )
   (wire (pts (xy 120.65 187.96) (xy 135.255 187.96))
     (stroke (width 0) (type default) (color 0 0 0 0))
@@
     (stroke (width 0) (type default) (color 0 0 0 0))
   )
-  (wire (pts (xy 281.305 57.15) (xy 281.305 59.055))
+  (wire (pts (xy 281.94 57.15) (xy 281.94 59.055))
     (stroke (width 0) (type default) (color 0 0 0 0))
   )
@@
     (stroke (width 0) (type default) (color 0 0 0 0))
   )
-  (wire (pts (xy 80.01 133.985) (xy 80.01 131.445))
+  (wire (pts (xy 80.01 130.81) (xy 80.01 133.985))
     (stroke (width 0) (type default) (color 0 0 0 0))
   )
@@
     (stroke (width 0) (type default) (color 0 0 0 0))
   )
-  (wire (pts (xy 276.86 57.15) (xy 281.305 57.15))
+  (wire (pts (xy 276.86 57.15) (xy 281.94 57.15))
     (stroke (width 0) (type default) (color 0 0 0 0))
   )
@@
     (stroke (width 0) (type default) (color 0 0 0 0))
   )
-  (wire (pts (xy 281.305 57.15) (xy 281.305 55.245))
+  (wire (pts (xy 281.94 52.07) (xy 281.94 57.15))
     (stroke (width 0) (type default) (color 0 0 0 0))
   )
@@
     (stroke (width 0) (type default) (color 0 0 0 0))
   )
-  (wire (pts (xy 27.94 131.445) (xy 27.94 135.255))
+  (wire (pts (xy 27.94 131.445) (xy 27.94 132.08))
     (stroke (width 0) (type default) (color 0 0 0 0))
   )
@@
     (stroke (width 0) (type default) (color 0 0 0 0))
   )
+  (wire (pts (xy 27.94 132.08) (xy 27.94 135.255))
+    (stroke (width 0) (type default) (color 0 0 0 0))
+  )
   (wire (pts (xy 166.37 62.865) (xy 165.1 62.865))
     (stroke (width 0) (type default) (color 0 0 0 0))
@@
     (stroke (width 0) (type default) (color 0 0 0 0))
   )
+  (wire (pts (xy 22.86 132.08) (xy 27.94 132.08))
+    (stroke (width 0) (type default) (color 0 0 0 0))
+  )
   (wire (pts (xy 52.705 38.1) (xy 67.31 38.1))
-    (stroke (width 0) (type default) (color 0 0 0 0))
-  )
-  (wire (pts (xy 23.495 131.445) (xy 27.94 131.445))
-    (stroke (width 0) (type default) (color 0 0 0 0))
-  )
-  (wire (pts (xy 23.495 128.905) (xy 23.495 131.445))
     (stroke (width 0) (type default) (color 0 0 0 0))
   )
@@
       (effects (font (size 1.27 1.27)) hide)
     )
+  )
+  (symbol (lib_id "power:VDD") (at 281.94 52.07 0) (unit 1)
+    (in_bom yes) (on_board yes) (fields_autoplaced)
+    (property "Reference" "#PWR030" (id 0) (at 281.94 55.88 0)
+      (effects (font (size 1.27 1.27)) hide)
+    )
+    (property "Value" "VDD" (id 1) (at 281.94 46.99 0))
+    (property "Footprint" "" (id 2) (at 281.94 52.07 0)
+      (effects (font (size 1.27 1.27)) hide)
+    )
+    (property "Datasheet" "" (id 3) (at 281.94 52.07 0)
+      (effects (font (size 1.27 1.27)) hide)
+    )
+    (pin "1")
   )
   (symbol (lib_id "Device:C_Small") (at 27.94 137.795 0) (unit 1)
@@
     (pin "1")
   )
-  (symbol (lib_id "power:+4V") (at 281.305 55.245 0) (unit 1)
-    (in_bom yes) (on_board yes) (fields_autoplaced)
-    (property "Reference" "#PWR0104" (id 0) (at 281.305 59.055 0)
-      (effects (font (size 1.27 1.27)) hide)
-    )
-    (property "Value" "+4V" (id 1) (at 281.305 51.6405 0))
-    (property "Footprint" "" (id 2) (at 281.305 55.245 0)
-      (effects (font (size 1.27 1.27)) hide)
-    )
-    (property "Datasheet" "" (id 3) (at 281.305 55.245 0)
-      (effects (font (size 1.27 1.27)) hide)
-    )
-    (pin "1")
-  )
   (symbol (lib_id "power:GND") (at 64.135 118.745 0) (unit 1)
     (in_bom yes) (on_board yes) (fields_autoplaced)
@@
     (pin "2")
   )
-  (symbol (lib_id "Connector:TestPoint") (at 281.305 59.055 180) (unit 1)
-    (in_bom yes) (on_board yes)
-    (property "Reference" "TP3" (id 0) (at 281.5401 67.31 90)
+  (symbol (lib_id "Connector:TestPoint") (at 281.94 59.055 180) (unit 1)
+    (in_bom yes) (on_board yes)
+    (property "Reference" "TP3" (id 0) (at 282.1751 67.31 90)
       (effects (font (size 1.27 1.27)) (justify right))
     )
-    (property "Value" "TestPoint" (id 1) (at 278.765 67.31 90)
+    (property "Value" "TestPoint" (id 1) (at 279.4 67.31 90)
       (effects (font (size 1.27 1.27)) (justify right))
     )
-    (property "Footprint" "TestPoint:TestPoint_Pad_D1.0mm" (id 2) (at 276.225 59.055 0)
-      (effects (font (size 1.27 1.27)) hide)
-    )
-    (property "Datasheet" "~" (id 3) (at 276.225 59.055 0)
+    (property "Footprint" "TestPoint:TestPoint_Pad_D1.0mm" (id 2) (at 276.86 59.055 0)
+      (effects (font (size 1.27 1.27)) hide)
+    )
+    (property "Datasheet" "~" (id 3) (at 276.86 59.055 0)
       (effects (font (size 1.27 1.27)) hide)
     )
@@
     (pin "1")
     (pin "2")
-  )
-  (symbol (lib_id "power:+3V0") (at 80.01 131.445 0) (unit 1)
-    (in_bom yes) (on_board yes) (fields_autoplaced)
-    (property "Reference" "#PWR015" (id 0) (at 80.01 135.255 0)
-      (effects (font (size 1.27 1.27)) hide)
-    )
-    (property "Value" "+3V0" (id 1) (at 80.01 127.8405 0))
-    (property "Footprint" "" (id 2) (at 80.01 131.445 0)
-      (effects (font (size 1.27 1.27)) hide)
-    )
-    (property "Datasheet" "" (id 3) (at 80.01 131.445 0)
-      (effects (font (size 1.27 1.27)) hide)
-    )
-    (pin "1")
   )
   (symbol (lib_id "SamacSys_Parts:2N7002KDW_R1_00001") (at 166.37 60.325 0) (unit 1)
@@
     (pin "5")
   )
+  (symbol (lib_id "power:VDD") (at 22.86 125.73 0) (unit 1)
+    (in_bom yes) (on_board yes) (fields_autoplaced)
+    (property "Reference" "#PWR01" (id 0) (at 22.86 129.54 0)
+      (effects (font (size 1.27 1.27)) hide)
+    )
+    (property "Value" "VDD" (id 1) (at 22.86 120.65 0))
+    (property "Footprint" "" (id 2) (at 22.86 125.73 0)
+      (effects (font (size 1.27 1.27)) hide)
+    )
+    (property "Datasheet" "" (id 3) (at 22.86 125.73 0)
+      (effects (font (size 1.27 1.27)) hide)
+    )
+    (pin "1")
+  )
   (symbol (lib_id "power:GND") (at 27.94 142.875 0) (unit 1)
     (in_bom yes) (on_board yes) (fields_autoplaced)
@@
     (pin "1")
   )
-  (symbol (lib_id "power:+4V") (at 23.495 128.905 0) (unit 1)
-    (in_bom yes) (on_board yes) (fields_autoplaced)
-    (property "Reference" "#PWR01" (id 0) (at 23.495 132.715 0)
-      (effects (font (size 1.27 1.27)) hide)
-    )
-    (property "Value" "+4V" (id 1) (at 23.495 125.3005 0))
-    (property "Footprint" "" (id 2) (at 23.495 128.905 0)
-      (effects (font (size 1.27 1.27)) hide)
-    )
-    (property "Datasheet" "" (id 3) (at 23.495 128.905 0)
-      (effects (font (size 1.27 1.27)) hide)
-    )
-    (pin "1")
-  )
   (symbol (lib_id "power:GND") (at 25.4 71.755 0) (unit 1)
     (in_bom yes) (on_board yes) (fields_autoplaced)
@@
     )
     (property "Datasheet" "" (id 3) (at 280.035 134.62 0)
+      (effects (font (size 1.27 1.27)) hide)
+    )
+    (pin "1")
+  )
+  (symbol (lib_id "power:+4V") (at 80.01 130.81 0) (unit 1)
+    (in_bom yes) (on_board yes) (fields_autoplaced)
+    (property "Reference" "#PWR015" (id 0) (at 80.01 134.62 0)
+      (effects (font (size 1.27 1.27)) hide)
+    )
+    (property "Value" "+4V" (id 1) (at 80.01 127.2055 0))
+    (property "Footprint" "" (id 2) (at 80.01 130.81 0)
+      (effects (font (size 1.27 1.27)) hide)
+    )
+    (property "Datasheet" "" (id 3) (at 80.01 130.81 0)
       (effects (font (size 1.27 1.27)) hide)
     )
@@
   )
   (symbol_instances
-    (path "/ba1b232e-349c-412e-8bd5-d09fd9db5a13"
-      (reference "#PWR01") (unit 1) (value "+4V") (footprint "")
+    (path "/a2f0b1d5-c140-4324-a09a-cbfffd026259"
+      (reference "#PWR01") (unit 1) (value "VDD") (footprint "")
     )
     (path "/a4795988-d1b1-45e0-98cd-aeeb4c0b8960"
@@
       (reference "#PWR014") (unit 1) (value "GND") (footprint "")
     )
-    (path "/8b2fc0eb-af5c-404f-b3f2-7d77ced4c2dd"
-      (reference "#PWR015") (unit 1) (value "+3V0") (footprint "")
+    (path "/da1d78a3-1a4b-488d-ab03-33feddcbc27f"
+      (reference "#PWR015") (unit 1) (value "+4V") (footprint "")
     )
     (path "/900e80f3-48a3-4549-ad6a-555a53fe6e3b"
@@
       (reference "#PWR029") (unit 1) (value "GND") (footprint "")
     )
+    (path "/0de44de0-4280-4bf4-b80f-f93aa5f680a5"
+      (reference "#PWR030") (unit 1) (value "VDD") (footprint "")
+    )
     (path "/d92bd81c-a4ef-4905-a738-66f88d689309"
       (reference "#PWR032") (unit 1) (value "+5V") (footprint "")
@@
       (reference "#PWR0103") (unit 1) (value "+BATT") (footprint "")
     )
-    (path "/7d9e3797-b6ee-453e-ae2a-ebdccaf33ce8"
-      (reference "#PWR0104") (unit 1) (value "+4V") (footprint "")
-    )
     (path "/d4265251-5371-423a-be0b-550112080266"
