File: SNAP Project PCB Files/PCB Files V6.0/SNAP_Project.kicad_pcb (KiCad board)
At the start: 4 copper layers, 66.7 x 47.2 mm, 109 parts, among them IC1 ADP121-AUJZ30R7, IC2 STM32WB35CCU7A, J1 USB_C_Receptacle_USB2.0, J3 Serial Wire Debug, J4 OLED Screen Conn, Q1 2N7000, Q2 2N7000, Q3 2N7000, Q4 SFH 310, Q5 2N7002KDW_R1_00001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

Commit message: Last Commit before production
Parts:
- R3: footprint Resistor_SMD:R_0603_1608Metric -> Resistor_SMD:R_0805_2012Metric
- moved D2 0.53 mm to (71.3, 99.3)
- moved R3 0.30 mm to (75.2, 97.0)
Routing:
- net WP7_EN: track 68.6 -> 68.1 mm
Other:
- board text added: "Design by: L. Zagastizabal"
